File: amplifier/amplifier.kicad_sch (KiCad schematic)
At the start: 6 parts

Commit message: update amplifier
Parts:
- removed Q?: Q_NPN_CBE, symbol Device:Q_NPN_CBE
- added J?: to fly, symbol Connector_Generic:Conn_01x02
- added J?: from ESP32, symbol Connector_Generic:Conn_01x04
- added Q? (x2): Q_NPN_Darlington_BCE, symbol Device:Q_NPN_Darlington_BCE
- added R? (x2): 3k, symbol Device:R
- added U? (x3): LM358, symbol Amplifier_Operational:LM358
- J?: value Conn_01x03_Male -> enable/disable system
- J?: value Conn_01x02_Female -> from power supply
- R?: value 30k -> 60k
Connections:
- net GND: now also J?.4 (Pin_4), Q?.3 (E), U?.3 (+), U?.4 (V-)
- net Vin: now also Q?.1 (B)
- net Vout: now also J?.1 (Pin_1), Q?.2 (C)
- net at R?.1: now also Q?.3 (E)
- new net: R?.1, R?.2, U?.2 (-)
- new net: Q?.1 (B), R?.2, U?.1
- new net: J?.2 (Pin_2), Q?.2 (C)
- new net: J?.1 (Pin_1), R?.1
- new net +5V: J?.3 (Pin_3), U?.8 (V+)
- no-connect marks 0 -> 4
Other:
- moved on the sheet: J?, R?

Commit message: update amplifier
Parts:
- added R?: 270, symbol Device:R
Connections:
- net at J?.2 (Pin_2): now also R?.1
- net Vin: no longer names the net of Q?.1 (B)
- net Vin: now also R?.2
- no-connect marks 4 -> 3
Changed lines of the file:
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@@
   (junction (at 152.146 83.566) (diameter 0) (color 0 0 0 0)
   )
-  (no_connect (at 112.014 72.898))
   (no_connect (at 132.08 133.35))
   (no_connect (at 116.84 135.89))
@@
     (stroke (width 0) (type default) (color 0 0 0 0))
   )
+  (wire (pts (xy 124.714 107.442) (xy 253.492 107.442))
+    (stroke (width 0) (type default) (color 0 0 0 0))
+  )
   (wire (pts (xy 127.762 83.566) (xy 142.494 83.566))
     (stroke (width 0) (type default) (color 0 0 0 0))
@@
     (stroke (width 0) (type default) (color 0 0 0 0))
   )
+  (wire (pts (xy 253.492 107.442) (xy 253.492 79.756))
+    (stroke (width 0) (type default) (color 0 0 0 0))
+  )
   (wire (pts (xy 154.432 139.954) (xy 154.432 142.494))
     (stroke (width 0) (type default) (color 0 0 0 0))
@@
     (stroke (width 0) (type default) (color 0 0 0 0))
   )
+  (wire (pts (xy 112.014 72.898) (xy 124.714 72.898))
+    (stroke (width 0) (type default) (color 0 0 0 0))
+  )
   (wire (pts (xy 171.704 81.026) (xy 178.308 81.026))
     (stroke (width 0) (type default) (color 0 0 0 0))
@@
     (stroke (width 0) (type default) (color 0 0 0 0))
   )
+  (wire (pts (xy 253.492 68.326) (xy 253.238 68.326))
+    (stroke (width 0) (type default) (color 0 0 0 0))
+  )
+  (wire (pts (xy 124.714 72.898) (xy 124.714 107.442))
+    (stroke (width 0) (type default) (color 0 0 0 0))
+  )
   (wire (pts (xy 154.432 122.174) (xy 154.432 124.714))
     (stroke (width 0) (type default) (color 0 0 0 0))
   )
-  (wire (pts (xy 253.238 66.802) (xy 253.238 72.898))
+  (wire (pts (xy 253.492 72.136) (xy 253.492 68.326))
     (stroke (width 0) (type default) (color 0 0 0 0))
   )
@@
     (stroke (width 0) (type default) (color 0 0 0 0))
   )
-  (wire (pts (xy 253.238 72.898) (xy 250.444 72.898))
-    (stroke (width 0) (type default) (color 0 0 0 0))
-  )
   (wire (pts (xy 178.308 81.026) (xy 178.308 80.772))
     (stroke (width 0) (type default) (color 0 0 0 0))
@@
   )
   (wire (pts (xy 203.2 41.656) (xy 203.2 36.322))
+    (stroke (width 0) (type default) (color 0 0 0 0))
+  )
+  (wire (pts (xy 253.238 66.802) (xy 253.238 68.326))
     (stroke (width 0) (type default) (color 0 0 0 0))
   )
@@
     )
   )
-  (global_label "Vin" (shape input) (at 250.444 72.898 180) (fields_autoplaced)
-    (effects (font (size 1.27 1.27)) (justify right))
-    (property "Intersheet References" "${INTERSHEET_REFS}" (id 0) (at 245.1885 72.8186 0)
-      (effects (font (size 1.27 1.27)) (justify right) hide)
-    )
-  )
   (symbol (lib_id "Amplifier_Operational:LM358") (at 124.46 133.35 0) (unit 2)
     (in_bom yes) (on_board yes) (fields_autoplaced)
@@
     (pin "2")
   )
+  (symbol (lib_id "Device:R") (at 253.492 75.946 180) (unit 1)
+    (in_bom yes) (on_board yes) (fields_autoplaced)
+    (property "Reference" "R?" (id 0) (at 255.27 75.1113 0)
+      (effects (font (size 1.27 1.27)) (justify right))
+    )
+    (property "Value" "270" (id 1) (at 255.27 77.6482 0)
+      (effects (font (size 1.27 1.27)) (justify right))
+    )
+    (property "Footprint" "" (id 2) (at 255.27 75.946 90)
+      (effects (font (size 1.27 1.27)) hide)
+    )
+    (property "Datasheet" "~" (id 3) (at 253.492 75.946 0)
+      (effects (font (size 1.27 1.27)) hide)
+    )
+    (pin "1")
+    (pin "2")
+  )
   (symbol (lib_id "power:GND") (at 204.47 100.838 0) (unit 1)
     (in_bom yes) (on_board yes) (fields_autoplaced)
@@
       (reference "R?") (unit 1) (value "3k") (footprint "")
     )
+    (path "/59d21793-df1b-4037-a9be-9dc30aa6db0e"
+      (reference "R?") (unit 1) (value "270") (footprint "")
+    )
     (path "/91bab05a-eac7-4838-ac4d-d89e94de4f84"
